File: Hw/batteryCharger.sch (KiCad schematic (older format))
At the start: 13 parts, among them J1 Vcc, J2 GND, J3 BAT, J4 GND, U1 MCP73831-2-OT

Commit message: Update schematic
Parts:
- added R4: 2.5K, Resistor_SMD:R_0805_2012Metric_Pad1.15x1.40mm_HandSolder, symbol Device:R
Connections:
- net at R2.2, U1.5 (PROG): now also R4.2; no longer JP1.1
- new net: JP1.1, R4.1
Other:
- moved on the sheet: JP1
Changed lines of the file:
@@
 L Device:Jumper_NO_Small JP1
 U 1 1 5D238183
-P 5070 3725
-F 0 "JP1" V 5024 3773 50  0000 L CNN
-F 1 "JP1" V 5115 3773 50  0000 L CNN
-F 2 "" H 5070 3725 50  0001 C CNN
-F 3 "~" H 5070 3725 50  0001 C CNN
-	1    5070 3725
+P 5070 4095
+F 0 "JP1" V 5024 4143 50  0000 L CNN
+F 1 "JP1" V 5115 4143 50  0000 L CNN
+F 2 "" H 5070 4095 50  0001 C CNN
+F 3 "~" H 5070 4095 50  0001 C CNN
+	1    5070 4095
 	0    1    1    0
 $EndComp
@@
 L power:GND #PWR011
 U 1 1 5D23A033
-P 5070 3950
-F 0 "#PWR011" H 5070 3700 50  0001 C CNN
-F 1 "GND" H 5075 3777 50  0000 C CNN
-F 2 "" H 5070 3950 50  0001 C CNN
-F 3 "" H 5070 3950 50  0001 C CNN
-	1    5070 3950
+P 5070 4320
+F 0 "#PWR011" H 5070 4070 50  0001 C CNN
+F 1 "GND" H 5075 4147 50  0000 C CNN
+F 2 "" H 5070 4320 50  0001 C CNN
+F 3 "" H 5070 4320 50  0001 C CNN
+	1    5070 4320
 	1    0    0    -1
 $EndComp
 Wire Wire Line
-	5070 3950 5070 3825
+	5070 4320 5070 4195
+$Comp
+L Device:R R4
+U 1 1 5D36C008
+P 5070 3775
+F 0 "R4" H 5000 3729 50  0000 R CNN
+F 1 "2.5K" H 5000 3820 50  0000 R CNN
+F 2 "Resistor_SMD:R_0805_2012Metric_Pad1.15x1.40mm_HandSolder" V 5000 3775 50  0001 C CNN
+F 3 "~" H 5070 3775 50  0001 C CNN
+F 4 "CR0805-FX-2491ELF" H 5070 3775 50  0001 C CNN "manf#"
+	1    5070 3775
+	-1   0    0    1
+$EndComp
+Wire Wire Line
+	5070 3925 5070 3995
 $EndSCHEMATC
